File: StreetSweeper/StreetSweeper.sch (KiCad schematic (older format))
At the start: 14 parts, among them J1 Dist Sensor, J10 M3, J11 M2, J12 M4, J2 Bluetooth, J9 M1, P1 Power, P2 Analog, P3 Digital, P4 Digital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

Commit message: schematic done.
Parts:
- added F_1: Conn_01x04_Female, symbol Connector:Conn_01x04_Female
- added U2: TB6612F, symbol 2xx_ence_uc_kicad5:TB6612F
- J1, J2: symbol Conn_01x04 -> Connector_Generic:Conn_01x04
- J10, P2: symbol CONN_01X06 -> Connector_Generic:Conn_01x06
- J11, P3: symbol CONN_01X10 -> Connector_Generic:Conn_01x10
- J12, J9, P1, P4: symbol CONN_01X08 -> Connector_Generic:Conn_01x08
- P5, P6, P7, P8: symbol CONN_01X01 -> Connector_Generic:Conn_01x01
Connections:
- net labels added: GND_9, PIN_7, VCC_9
- wire segments 86 -> 116
- no-connect marks 10 -> 12
Other:
- note removed: "Connections"
- moved on the sheet: J1, J2
