File: StreetSweeper/buzzerCircuit.sch (KiCad schematic (older format))
At the start: 15 parts

Commit message: schematic done.
Parts:
- added B1: Buzzer, Connector_PinHeader_2.54mm:PinHeader_1x02_P2.54mm_Vertical, symbol 2xx_ence_uc_kicad5:UC_Speaker
- added C3: 100u, symbol Device:CP1
- added C4: 1u, symbol Device:CP1
- added C5: 10u, symbol Device:CP1
- added R6: 100k, Resistors_THT:R_Axial_DIN0207_L6.3mm_D2.5mm_P2.54mm_Vertical, symbol 2xx_ence_uc_kicad5:UC_R
- B_1: renamed from J?; symbol UC_CONN_01X02 -> 2xx_ence_uc_kicad5:UC_CONN_01X02
- C1, C2: renamed from C?; value CP1 -> 1u; symbol CP1 -> Device:CP1
- D1: renamed from D?; symbol LED -> 2xx_ence_uc_kicad5:UC_LED
- D2, D3: renamed from D?; symbol UC_D_SCHOTTKY -> 2xx_ence_uc_kicad5:UC_D_SCHOTTKY
- Q1, Q2: renamed from Q?; symbol 2N3904 -> Transistor_BJT:2N3904
- Q3: renamed from Q?; value UC_Q_NMOS -> 2N5485; symbol UC_Q_NMOS -> 2xx_ence_uc_kicad5:UC_Q_NMOS
- R1, R4, R5: renamed from R?; value UC_R -> 330; symbol UC_R -> 2xx_ence_uc_kicad5:UC_R
- R2, R3: renamed from R?; value UC_R -> 4.7k; symbol UC_R -> 2xx_ence_uc_kicad5:UC_R
- U1: renamed from U?; value UC_LMC6462 -> LMC6462; symbol UC_LMC6462 -> 2xx_ence_uc_kicad5:UC_LMC6462
Connections:
- net GND: now also B1.2, C4.2
- net at Q3.3 (S), U1.2 (-): now also C3.1, R6.2
- net at U1.1: now also C3.2, C4.1, C5.1, R6.1
- net GND_2 renamed VCC_9
- net Pin7 renamed PIN_7
- net VCC_2 renamed GND_9
- new net: B1.1, C5.2
Other:
- moved on the sheet: B_1, C1, C2, D2, D3, Q1, Q2, Q3, R1, R2, R3, R4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
